File: rm_foc_driver.kicad_sch (KiCad schematic)
At the start: 88 parts, among them J1 SWD, J2 TMC4671, J3 UART, J4 TMC4671, J5 Conn_01x03, J6 Conn_01x02, J8 Conn_01x03, Q1 CSD18540Q5B, Q2 CSD18540Q5B, Q3 CSD18540Q5B, Q4 CSD18540Q5B, Q5 CSD18540Q5B, Q6 CSD18540Q5B, U1 TPS54540, U10 74HC244, U2 RT9013, U3 STM32F401CCUx, U4 SY8303, U5 IR2104, U6 INA2180, U7 MT6701, U8 IR2104, U9 IR2104, Y1 Crystal_GND24

Commit message: remove mcu...
Parts:
- removed C11, C9: 22pF, Capacitor_SMD:C_0603_1608Metric, symbol Device:C
- removed C15, C16, C2, C20: 1uF, Capacitor_SMD:C_0603_1608Metric, symbol Device:C
- removed C22: C_Polarized, Capacitor_SMD:CP_Elec_4x5.4, symbol Device:C_Polarized
- removed C24, C33: 10uF, Capacitor_SMD:C_0805_2012Metric, symbol Device:C
- removed C34, C35, C36, C37, C4: 100nF, Capacitor_SMD:C_0603_1608Metric, symbol Device:C
- removed C6: 4.7uF, Capacitor_SMD:C_0603_1608Metric, symbol Device:C
- removed D1, D2: LED, LED_SMD:LED_0603_1608Metric, symbol Device:LED
- removed J1: SWD, Connector_PinHeader_2.54mm:PinHeader_1x04_P2.54mm_Horizontal, symbol Connector_Generic:Conn_01x04
- removed J3: UART, Connector_PinHeader_2.54mm:PinHeader_1x04_P2.54mm_Horizontal, symbol Connector_Generic:Conn_01x04
- removed J4: TMC4671, Connector_PinHeader_2.54mm:PinHeader_1x04_P2.54mm_Vertical, symbol Connector_Generic:Conn_01x04
- removed R1, R3, R4, R5: 10k, Resistor_SMD:R_0603_1608Metric, symbol Device:R
- removed U2: RT9013, Package_TO_SOT_SMD:SOT-23-5, symbol Interface_Ethernet:RT9013
- removed U3: STM32F401CCUx, Package_DFN_QFN:QFN-48-1EP_7x7mm_P0.5mm_EP5.6x5.6mm, symbol MCU_ST_STM32F4:STM32F401CCUx
- removed U6: INA2180, Package_SO:VSSOP-8_3.0x3.0mm_P0.65mm, symbol Amplifier_Current:INA2180
- removed U7: MT6701, Package_SO:SOP-8_3.9x4.9mm_P1.27mm, symbol Sensor_Magnetic:MT6701
- removed Y1: Crystal_GND24, Crystal:Crystal_SMD_3225-4Pin_3.2x2.5mm, symbol Device:Crystal_GND24
- added C23: 100nF, Capacitor_SMD:C_0603_1608Metric, symbol Device:C
- added R10, R9: 2.5k, Resistor_SMD:R_0603_1608Metric, symbol Device:R
- added U6, U7: LM236, Package_SO:PowerIntegrations_SO-8, symbol My_lib:LM236
- added U8, U9: INA199, Package_TO_SOT_SMD:SOT-363_SC-70-6_Handsoldering, symbol My_lib:INA199
- C2: renamed from C23; value 47uF -> 100nF; footprint Capacitor_SMD:C_0805_2012Metric -> Capacitor_SMD:C_0603_1608Metric
- renumbered C3 to C1, C13 to C10, C14 to C11, C17 to C12, C18 to C13, C21 to C14, C25 to C16, C26 to C17, C27 to C18, C29 to C19, C30 to C20, C31 to C21, C32 to C22, C5 to C3, C1 to C4, C7 to C5, C19 to C6, C8 to C7, C10 to C8, C12 to C9, D3 to D1, D4 to D2, D5 to D3, D6 to D4, J2 to J1, J6 to J2, J8 to J3, J5 to J4, L2 to L1, L1 to L2, R2 to R1, R9 to R11, R10 to R17, R11 to R18, R17 to R2, R18 to R3, R6 to R4, R19 to R5, R20 to R6, U4 to U2, U5 to U3, U8 to U4, U9 to U5
Connections:
- net +5V: now also C23.1, R10.1, R9.1, U8.3 (VCC), U9.3 (VCC)
- net GND: now also Q2.1 (S), Q2.2 (S), Q2.3 (S), Q4.1 (S), Q4.2 (S), Q4.3 (S), C23.2, U6.4 (ANODE), U7.4 (ANODE), U8.2 (GND), U9.2 (GND); no longer R17.2, R18.2
- net SH_A: now also J3.3 (Pin_3), R17.1, U8.5 (IN-); no longer J3.1 (Pin_1), Q1.1 (S), Q1.2 (S), Q1.3 (S), Q2.5 (D)
- net SH_B: now also J3.1 (Pin_1), R18.1, U9.5 (IN-); no longer J3.2 (Pin_2), Q3.1 (S), Q3.2 (S), Q3.3 (S), Q4.5 (D)
- net SH_C: now also J3.2 (Pin_2); no longer J3.3 (Pin_3)
- net SO1: now also U8.6 (OUT)
- net SO2: now also U9.6 (OUT)
- removed net SL_A: Q2.1 (S), Q2.2 (S), Q2.3 (S), R17.1
- removed net SL_B: Q4.1 (S), Q4.2 (S), Q4.3 (S), R18.1
- new net: R9.2, U6.8 (CATHODE), U8.1 (REF)
- new net: R10.2, U7.8 (CATHODE), U9.1 (REF)
- new net A_P: Q1.1 (S), Q1.2 (S), Q1.3 (S), Q2.5 (D), R17.2, U8.4 (IN+)
- new net B_P: Q3.1 (S), Q3.2 (S), Q3.3 (S), Q4.5 (D), R18.2, U9.4 (IN+)
- no-connect marks 37 -> 14
Other:
- note removed: "3.3V LDO"
- note removed: "MCU"
- note removed: "POSITION SENSOR"
- moved on the sheet: C2, J1, J2, J3, J4, R17, R18

Commit message: 20230111 AD8418
Parts:
- removed R10, R9: 2.5k, Resistor_SMD:R_0603_1608Metric, symbol Device:R
- removed U6, U7: LM236, Package_SO:PowerIntegrations_SO-8, symbol My_lib:LM236
- removed U8, U9: INA199, Package_TO_SOT_SMD:SOT-363_SC-70-6_Handsoldering, symbol My_lib:INA199
- added U6, U7: AD8418, Package_SO:SOP-8_3.9x4.9mm_P1.27mm, symbol Amplifier_Current:AD8418
Connections:
- net +5V: now also U6.6 (VS), U6.7 (REF1), U7.6 (VS), U7.7 (REF1)
- net A_P: now also U7.8 (IN+)
- net B_P: now also U6.8 (IN+)
- net GND: now also U6.2 (GND), U6.3 (REF2), U7.2 (GND), U7.3 (REF2)
- net SH_A: now also U7.1 (IN-)
- net SH_B: now also U6.1 (IN-)
- net SO1: now also U7.5 (OUT)
- net SO2: now also U6.5 (OUT)
- no-connect marks 14 -> 12
